Commit message: added launch file and changes in urdf

File: matrix_bot/urdf/Matrix_bot.urdf (robot description, URDF)
Before this commit: robot Matrix_bot, 7 links, 6 joints
Links:
- link base_link: geometry collision mesh filename=package://matrix_bot/meshes/base_link.STL; visual mesh filename=package://matrix_bot/meshes/base_link.STL
- link camera: geometry collision mesh filename=package://matrix_bot/meshes/camera.STL; visual mesh filename=package://matrix_bot/meshes/camera.STL
- link castor_wheel: geometry collision mesh filename=package://matrix_bot/meshes/castor_wheel.STL; visual mesh filename=package://matrix_bot/meshes/castor_wheel.STL
- link imu_sensor: geometry collision mesh filename=package://matrix_bot/meshes/imu_sensor.STL; visual mesh filename=package://matrix_bot/meshes/imu_sensor.STL
- link left_wheel: geometry collision mesh filename=package://matrix_bot/meshes/left_wheel.STL; visual mesh filename=package://matrix_bot/meshes/left_wheel.STL
- link lidar_sensor: geometry collision mesh filename=package://matrix_bot/meshes/lidar_sensor.STL; visual mesh filename=package://matrix_bot/meshes/lidar_sensor.STL
- link right_wheel: geometry collision mesh filename=package://matrix_bot/meshes/right_wheel.STL; visual mesh filename=package://matrix_bot/meshes/right_wheel.STL
Joints:
- joint castor_wheel_joint: type continuous -> fixed

Commit message: some changes

File: matrix_bot/urdf/Matrix_bot.urdf (robot description, URDF)
Before this commit: robot Matrix_bot, 7 links, 6 joints
Links:
- link base_link: mass 0.13905 -> 2.0
- link camera: mass 0.0014912 -> 0.1
- link castor_wheel: mass 0.050965 -> 0.2
- link imu_sensor: mass 0.001935 -> 0.1
- link left_wheel: mass 0.029452 -> 0.2
- link lidar_sensor: mass 0.0070686 -> 0.1
- link right_wheel: mass 0.029452 -> 0.2
Joints:
- joint castor_wheel_joint: axis 0.24121 -0.92049 -0.30745 -> 0 0 0
