Commit message: gazebo controller plugin

File: matrix_bot/urdf/gazebo_references_plugins.xacro (robot description, xacro)
@@ -12,25 +12,8 @@
   </material>
   <gazebo reference="base_link">
-    <material>base_blue</material>
+    <material>Gazebo/SkyBlue</material>
   </gazebo>
   <gazebo reference="left_wheel">
-    <material>wheel_black</material>
-  </gazebo>
-  <gazebo reference="right_wheel">
-    <material>wheel_black</material>
-  </gazebo>
-  <gazebo reference="castor">
-    <material>light_grey</material>
-  </gazebo>
-  <gazebo reference="imu">
-    <material>light_grey</material>
-  </gazebo>
-  <gazebo reference="lidar">
-    <material>light_grey</material>
-  </gazebo>
-  <gazebo reference="camera">
-    <material>light_grey</material>
-  </gazebo>
-  <gazebo reference="left_wheel">
+    <material>Gazebo/Black</material>
     <mu>1.0</mu>
     <mu2>1.0</mu2>
@@ -39,4 +22,5 @@
   </gazebo>
   <gazebo reference="right_wheel">
+    <material>Gazebo/Black</material>
     <mu>1.0</mu>
     <mu2>1.0</mu2>
@@ -44,3 +28,15 @@
     <kd>1.0</kd>
   </gazebo>
+  <gazebo reference="castor">
+    <material>Gazebo/Grey</material>
+  </gazebo>
+  <gazebo reference="imu">
+    <material>Gazebo/Green</material>
+  </gazebo>
+  <gazebo reference="lidar">
+    <material>Gazebo/Black</material>
+  </gazebo>
+  <gazebo reference="camera">
+    <material>Gazebo/Grey</material>
+  </gazebo>
 </robot>
