Commit message: updated reference

File: matrix_bot/urdf/gazebo_references_plugins.xacro (robot description, xacro)
@@ -14,20 +14,24 @@
     <material>Gazebo/SkyBlue</material>
   </gazebo>
-  <gazebo reference="left_wheel">
-    <material>Gazebo/Black</material>
-    <mu>1.0</mu>
-    <mu2>1.0</mu2>
-    <kp>1e6</kp>
-    <kd>1.0</kd>
-  </gazebo>
-  <gazebo reference="right_wheel">
-    <material>Gazebo/Black</material>
-    <mu>1.0</mu>
-    <mu2>1.0</mu2>
-    <kp>1e6</kp>
-    <kd>1.0</kd>
-  </gazebo>
+<gazebo reference="left_wheel">
+  <material>Gazebo/Black</material>
+  <mu1>1.0</mu1>    <!-- keep forward traction high -->
+  <mu2>0.15</mu2> <!-- let the wheel scrub sideways during turns -->
+  <kp>1e6</kp>
+  <kd>100.0</kd>
+  <fdir1>1 0 0</fdir1>  <!-- pin the friction direction explicitly -->
+</gazebo>
+<gazebo reference="right_wheel">
+  <material>Gazebo/Black</material>
+  <mu1>1.0</mu1>
+  <mu2>0.15</mu2>
+  <kp>1e6</kp>
+  <kd>100.0</kd>
+  <fdir1>1 0 0</fdir1>
+</gazebo>
   <gazebo reference="castor">
     <material>Gazebo/Grey</material>
+    <mu1 value="0.001"/>
+    <mu2 value="0.001"/>
   </gazebo>
   <gazebo reference="imu">

File: matrix_bot/urdf/gazebo_ros2_control.xacro (robot description, xacro)
@@ -20,13 +20,16 @@
             <left_joint>left_wheel_joint</left_joint>
             <right_joint>right_wheel_joint</right_joint>
-            <wheel_separation>0.1</wheel_separation>
+            <wheel_separation>0.115</wheel_separation>
             <wheel_diameter>0.05</wheel_diameter>
+            <max_wheel_torque>5.0</max_wheel_torque>
+            <max_wheel_acceleration>1.0</max_wheel_acceleration>
             <command_topic>cmd_vel</command_topic>
+            <cmd_vel_timeout>0.2</cmd_vel_timeout>
             <publish_odom>true</publish_odom>
-            <publish_odom_tf>true</publish_odom_tf>
+            <publish_odom_tf>false</publish_odom_tf>
             <odometry_topic>odom</odometry_topic>
             <odometry_frame>odom</odometry_frame>
             <robot_base_frame>base_link</robot_base_frame>
-            <publish_tf>true</publish_tf>
+            <publish_tf>false</publish_tf>
         </plugin>
     </gazebo>

File: matrix_bot/urdf/imu_plugin.xacro (robot description, xacro)
@@ -1,16 +1,65 @@
 <?xml version="1.0"?>
-<robot xmlns:xacro="http://www.ros.org/wiki/xacro" >
+<robot xmlns:xacro="http://www.ros.org/wiki/xacro">
+    <gazebo reference="imu_joint">
+        <preserveFixedJoint>true</preserveFixedJoint>
+        <disableFixedJointLumping>true</disableFixedJointLumping>
+    </gazebo>
     <gazebo reference="imu">
         <sensor name="imu_sensor" type="imu">
+            <!-- 1. Mandatory to keep the sensor publishing continuously -->
+            <always_on>true</always_on>
             <update_rate>50</update_rate>
+            <visualize>true</visualize>
             <pose>0 0 0 0 0 0</pose>
-            <visualize>true</visualize>
+            <!-- 2. Noise model (ROS 2 standard) -->
+            <imu>
+                <angular_velocity>
+                    <x>
+                        <noise type="gaussian">
+                            <mean>0.0</mean>
+                            <stddev>0.0001</stddev>
+                        </noise>
+                    </x>
+                    <y>
+                        <noise type="gaussian">
+                            <mean>0.0</mean>
+                            <stddev>0.0001</stddev>
+                        </noise>
+                    </y>
+                    <z>
+                        <noise type="gaussian">
+                            <mean>0.0</mean>
+                            <stddev>0.0001</stddev>
+                        </noise>
+                    </z>
+                </angular_velocity>
+                <linear_acceleration>
+                    <x>
+                        <noise type="gaussian">
+                            <mean>0.0</mean>
+                            <stddev>0.0001</stddev>
+                        </noise>
+                    </x>
+                    <y>
+                        <noise type="gaussian">
+                            <mean>0.0</mean>
+                            <stddev>0.0001</stddev>
+                        </noise>
+                    </y>
+                    <z>
+                        <noise type="gaussian">
+                            <mean>0.0</mean>
+                            <stddev>0.0001</stddev>
+                        </noise>
+                    </z>
+                </linear_acceleration>
+            </imu>
+            <!-- 3. Correct ROS 2 IMU plugin -->
             <plugin name="imu_plugin" filename="libgazebo_ros_imu_sensor.so">
                 <ros>
-                    <remapping>imu_plugin/imu:=imu/data</remapping>
+                    <namespace>/</namespace>
+                    <remapping>~/out:=/imu/data</remapping>
                 </ros>
-                <topic_name>imu/data</topic_name>
-                <frame_name>imu</frame_name>
-                <gaussian_noise>0.0001</gaussian_noise>
+                <initial_orientation_as_reference>false</initial_orientation_as_reference>
             </plugin>
         </sensor>

File: matrix_bot/urdf/lidar_plugin.xacro (robot description, xacro)
@@ -9,8 +9,8 @@
                 <scan>
                     <horizontal>
-                    <samples>720</samples>
+                    <samples>360</samples>
                     <resolution>1</resolution>
-                    <min_angle>-6.28</min_angle>
-                    <max_angle>6.28</max_angle>
+                    <min_angle>-3.14</min_angle>
+                    <max_angle>3.14</max_angle>
                     </horizontal>
                 </scan>
