Commit message: added imu plugin

File: matrix_bot/urdf/imu_plugin.xacro (robot description, xacro)
@@ -1,4 +1,4 @@
 <?xml version="1.0"?>
-<xacro:macro name="imu_plugin" params="">
+<robot xmlns:xacro="http://www.ros.org/wiki/xacro" >
     <gazebo reference="imu">
         <sensor name="imu_sensor" type="imu">
@@ -16,3 +16,3 @@
         </sensor>
     </gazebo>
-</xacro:macro>``
+</robot>
